Commit message: delet fdir

File: my_robot_description/urdf/robot.urdf.xacro (robot description, xacro)
@@ -30,6 +30,6 @@
     <color rgba="1 0 0 1"/>
   </material>
-<!-- WHEEL MACRO WITH FDIR -->
-  <xacro:macro name="wheel" params="name x y z fdir">
+<!-- WHEEL MACRO -->
+  <xacro:macro name="wheel" params="name x y z ">
     <link name="${name}_link">
       <visual>
@@ -52,11 +52,4 @@
       </inertial>
     </link>
-    <gazebo reference="${name}_link">
-      <mu1>1.0</mu1>
-      <mu2>0.0</mu2>
-      <fdir1>${fdir}</fdir1>
-      <kp>1e6</kp>
-      <kd>100.0</kd>
-    </gazebo>
     <joint name="${name}_joint" type="continuous">
       <parent link="base_link"/>
@@ -148,7 +141,7 @@
   </gazebo>
 <!-- X-Pattern Friction Directions -->
-  <xacro:wheel name="front_left_wheel"  x="0.2"  y="0.2"  z="-0.1" fdir="1 -1 0"/>
-  <xacro:wheel name="front_right_wheel" x="0.2"  y="-0.2" z="-0.1" fdir="1 1 0"/>
-  <xacro:wheel name="back_left_wheel"   x="-0.2" y="0.2"  z="-0.1" fdir="1 1 0"/>
-  <xacro:wheel name="back_right_wheel"  x="-0.2" y="-0.2" z="-0.1" fdir="1 -1 0"/>
+  <xacro:wheel name="front_left_wheel"  x="0.2"  y="0.2"  z="-0.1"/>
+  <xacro:wheel name="front_right_wheel" x="0.2"  y="-0.2" z="-0.1"/>
+  <xacro:wheel name="back_left_wheel"   x="-0.2" y="0.2"  z="-0.1"/>
+  <xacro:wheel name="back_right_wheel"  x="-0.2" y="-0.2" z="-0.1"/>
 </robot>
